File: HavenPCB.kicad_pcb (KiCad board)
At the start: 2 copper layers, 139.7 x 76.2 mm, 39 parts, among them J1 C52209111, SW1 BOOTSEL, U1 NCP1117ST33T3G, U2 RP2354A, U3 USBLC6-2SC6, Y1 ABM8-272-T3

Commit message: uwu nyaaa puurs at you
Parts:
- added C20: 4.7u, Capacitor_SMD:C_0402_1005Metric, F.Cu at (131.8, 86.3)
- added C21: 4.7u, Capacitor_SMD:C_0402_1005Metric, F.Cu at (128.0, 97.9)
- added C22: 4.7u, Capacitor_SMD:C_0402_1005Metric, F.Cu at (169.1, 39.0)
- added NT1: NetTie_2, NetTie:NetTie-2_SMD_Pad2.0mm, B.Cu at (151.9, 84.5)
- J1: value C52209111 -> C2765186; footprint easyeda2kicad:USB-SMD_HH-16P-TYPE-C-Y495 -> HavenPCB:USB-C-SMD_TYPE-C-16PIN-2MD-073
- moved TP6 78.8 mm to (179.4, 35.5)
- moved C13 72.1 mm to (166.3, 31.2)
- moved C14 72.1 mm to (166.3, 33.1)
- moved C18 69.1 mm to (169.1, 31.2)
- moved C19 69.1 mm to (169.1, 33.1)
- moved C10 62.8 mm to (163.4, 35.1)
- moved C8 62.8 mm to (163.4, 31.2)
- moved C12 62.8 mm to (163.4, 39.0)
- moved C15 60.0 mm to (166.3, 35.1)
- moved C16 60.0 mm to (166.3, 37.1)
- moved C17 60.0 mm to (166.3, 39.0)
- moved R1 42.4 mm to (155.0, 70.6), turned to -90 degrees
- moved R3 38.6 mm to (155.9, 88.9), turned to 180 degrees
- moved C5 38.2 mm to (155.9, 87.9)
- moved C4 36.2 mm to (148.3, 102.7), turned to 90 degrees
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Connections:
- net Net-(U2-USB_DM) renamed /RP_D-
- net Net-(U2-USB_DP) renamed /RP_D+
- C6 pad 2: GND -> VREG_GND
- C7 pad 2: GND -> VREG_GND
- U2 pad 47: GND -> VREG_GND
Routing:
- net VBUS: track 0.00 -> 43.9 mm, vias 0 -> 2
- net +1V1: track 0.00 -> 41.6 mm, vias 0 -> 4
- net +3V3: track 0.00 -> 37.4 mm, vias 0 -> 10
- net Net-(U2-XIN): track 0.00 -> 7.50 mm
- net /RP_D-: track 0.00 -> 6.80 mm
- net /RP_D+: track 0.00 -> 6.76 mm
- net Net-(J1-CC1): track 0.00 -> 6.66 mm
- net Net-(J1-CC2): track 0.00 -> 6.17 mm
- net /SWD: track 0.00 -> 5.78 mm
- net /USB_D+: track 0.00 -> 5.36 mm
- net /USB_D-: track 0.00 -> 5.22 mm
- net GND: track 0.00 -> 4.82 mm, vias 0 -> 19
- net /VREG_AVDD: track 0.00 -> 4.23 mm
- net Net-(R4-Pad1): track 0.00 -> 4.15 mm
- net Net-(C4-Pad2): track 0.00 -> 4.10 mm
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- added copper zone on In2.Cu, net +3V3
- added copper zone on B.Cu, net GND
- added copper zone on F.Cu, net GND
- added copper zone on In1.Cu, net GND
- added copper zone on B.Cu, net VREG_GND
Other:
- copper layers 2 -> 4
- board text added: "+3v3"
- board text added: "GND"
- board text added: "SWCLK"
- board text added: "SWD"
- board text added: "VBUS"

Commit message: dsafanjkhf
Parts:
- added SW2: Up, Button_Switch_THT:SW_PUSH_6mm_H5mm, F.Cu at (99.0, 86.9)
- added SW3: Right, Button_Switch_THT:SW_PUSH_6mm_H5mm, F.Cu at (114.0, 101.9)
- added SW4: Left, Button_Switch_THT:SW_PUSH_6mm_H5mm, F.Cu at (84.0, 101.9)
- added SW5: Down, Button_Switch_THT:SW_PUSH_6mm_H5mm, F.Cu at (99.0, 116.9)
- added SW6: X, Button_Switch_THT:SW_PUSH_6mm_H5mm, F.Cu at (186.7, 86.9)
- added SW7: Y, Button_Switch_THT:SW_PUSH_6mm_H5mm, F.Cu at (171.7, 101.9)
- added SW8: B, Button_Switch_THT:SW_PUSH_6mm_H5mm, F.Cu at (186.7, 116.9)
- added SW9: A, Button_Switch_THT:SW_PUSH_6mm_H5mm, F.Cu at (201.7, 101.9)
- moved C14 64.0 mm to (155.4, 96.2)
- moved C10 61.9 mm to (143.2, 93.7), turned to 180 degrees
- moved C13 61.2 mm to (156.1, 91.5)
- moved C12 60.7 mm to (146.3, 97.3), turned to 180 degrees
- moved C18 60.5 mm to (156.3, 90.3)
- moved C8 60.0 mm to (144.9, 88.2), turned to 90 degrees
- moved C15 58.4 mm to (156.1, 92.6)
- moved TP6 54.3 mm to (156.4, 84.7)
- moved C16 53.2 mm to (156.3, 89.3)
- moved C19 50.1 mm to (146.7, 77.9), turned to 180 degrees
- moved C17 49.8 mm to (148.6, 85.6), turned to 90 degrees
- moved C22 47.4 mm to (158.3, 85.2), turned to -90 degrees
- moved TP5 4.51 mm to (131.4, 82.8)
- moved C20 4.51 mm to (129.6, 82.4)
- moved C2 4.19 mm to (131.7, 95.5)
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Connections:
- U2 pad 13: unconnected-(U2-GPIO9-Pad13) -> /Down
- U2 pad 14: unconnected-(U2-GPIO10-Pad14) -> /Right
- U2 pad 32: unconnected-(U2-GPIO20-Pad32) -> /Y
- U2 pad 33: unconnected-(U2-GPIO21-Pad33) -> /B
- U2 pad 34: unconnected-(U2-GPIO22-Pad34) -> /A
- U2 pad 35: unconnected-(U2-GPIO23-Pad35) -> /X
- U2 pad 7: unconnected-(U2-GPIO4-Pad7) -> /Up
- U2 pad 8: unconnected-(U2-GPIO5-Pad8) -> /Left
Routing:
- net /Down: track 0.00 -> 70.0 mm
- net /Left: track 0.00 -> 68.5 mm
- net /A: track 0.00 -> 58.5 mm
- net /B: track 0.00 -> 57.7 mm
- net /Up: track 0.00 -> 49.2 mm
- net /Right: track 0.00 -> 47.0 mm
- net /X: track 0.00 -> 43.0 mm
- net /Y: track 0.00 -> 28.1 mm
- net +1V1: track 41.6 -> 28.0 mm
- net +3V3: track 37.4 -> 46.2 mm, vias 10 -> 12
- net VBUS: track 43.9 -> 42.2 mm
- net Net-(C4-Pad2): track 4.10 -> 3.35 mm
- net GND: track 4.82 -> 5.55 mm
- net /VREG_AVDD: track 4.23 -> 3.67 mm
- net VREG_GND: track 2.85 -> 3.38 mm
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- added copper zone on B.Cu, net +1V1
Other:
- board text added: "+1v1"

Commit message: final
Parts:
- removed C20, C21, C22: 4.7u, Capacitor_SMD:C_0402_1005Metric
- removed TP1, TP2, TP3, TP4, TP5, TP6: TestPoint, TestPoint:TestPoint_Pad_D1.5mm
- added G***: LOGO, LOGO, F.Cu at (146.9, 101.2)
- added G***: LOGO, LOGO, B.Cu at (146.8, 104.8)
- added REF**: MountingHole_3.2mm_M3, MountingHole:MountingHole_3.2mm_M3, F.Cu at (164.9, 71.1)
- added REF**: MountingHole_3.2mm_M3, MountingHole:MountingHole_3.2mm_M3, F.Cu at (134.9, 71.1)
Routing:
- net /SWD: track 5.78 -> 0.00 mm
- net +3V3: track 46.2 -> 41.7 mm
- net /SWCLK: track 3.76 -> 0.00 mm
- net +1V1: track 28.0 -> 24.3 mm
- net VBUS: track 42.2 -> 40.6 mm
- net /Left: track 68.5 -> 67.9 mm
Other:
- board text removed: "GND"
- board text removed: "SWCLK"
- board text removed: "SWD"
