File: HavenPCB.kicad_sch (KiCad schematic)
At the start: 33 parts, among them J1 C52209111, J2 JST, SW1 BOOTSEL, U1 RP2354A, U2 NCP1117ST33T3G, Y1 ABM8-272-T3

Commit message: jdasklfjlk
Parts:
- removed C19: 100n, symbol Device:C
- removed J2: JST, symbol Connector:Conn_01x03_Socket
- added C19: 100n, Capacitor_SMD:C_0402_1005Metric, symbol Device:C_Small
- added TP1, TP2, TP3, TP4, TP5, TP6: TestPoint, TestPoint:TestPoint_Pad_D1.5mm, symbol Connector:TestPoint
- added U3: USBLC6-2SC6, Package_TO_SOT_SMD:SOT-23-6, symbol Power_Protection:USBLC6-2SC6
- C1: renamed from C2; footprint (none) -> Capacitor_SMD:C_0402_1005Metric
- C10: renamed from C7; footprint (none) -> Capacitor_SMD:C_0402_1005Metric
- C11: renamed from C15; footprint (none) -> Capacitor_SMD:C_0402_1005Metric
- C12: renamed from C8; footprint (none) -> Capacitor_SMD:C_0402_1005Metric
- C13: renamed from C16; footprint (none) -> Capacitor_SMD:C_0402_1005Metric
- C14: renamed from C9; footprint (none) -> Capacitor_SMD:C_0402_1005Metric
- C15: renamed from C10; footprint (none) -> Capacitor_SMD:C_0402_1005Metric
- C16: renamed from C11; footprint (none) -> Capacitor_SMD:C_0402_1005Metric
- C17: renamed from C12; footprint (none) -> Capacitor_SMD:C_0402_1005Metric
- C18: renamed from C13; footprint (none) -> Capacitor_SMD:C_0402_1005Metric
- C2: renamed from C3; footprint (none) -> Capacitor_SMD:C_0402_1005Metric
- C3: renamed from C17; footprint (none) -> Capacitor_SMD:C_0402_1005Metric
- C4: renamed from C18; footprint (none) -> Capacitor_SMD:C_0402_1005Metric
- C5: renamed from C4; footprint (none) -> Capacitor_SMD:C_0402_1005Metric
- C6: renamed from C1; footprint (none) -> Capacitor_SMD:C_0402_1005Metric
- C7: renamed from C5; footprint (none) -> Capacitor_SMD:C_0402_1005Metric
- C8: renamed from C6; footprint (none) -> Capacitor_SMD:C_0402_1005Metric
- C9: renamed from C14; footprint (none) -> Capacitor_SMD:C_0402_1005Metric
- J1: footprint (none) -> easyeda2kicad:USB-SMD_HH-16P-TYPE-C-Y495
- L1: value 3.3U -> AOTA-B201610S3R3-101-T; footprint (none) -> Inductor_SMD:L_0805_2012Metric
- R1, R2, R3: footprint (none) -> Resistor_SMD:R_0402_1005Metric
- R4: renamed from R7; footprint (none) -> Resistor_SMD:R_0402_1005Metric
- R5: renamed from R4; footprint (none) -> Resistor_SMD:R_0402_1005Metric
- R6: renamed from R5; footprint (none) -> Resistor_SMD:R_0603_1608Metric
- R7: renamed from R6; footprint (none) -> Resistor_SMD:R_0603_1608Metric
- SW1: footprint (none) -> Button_Switch_SMD:SW_SPST_TS-1088-xR020
- Y1: footprint (none) -> Crystal:Crystal_SMD_3225-4Pin_3.2x2.5mm
- renumbered U2 to U1, U1 to U2
Connections:
- net +1V1: now also L1.2, U2.23 (DVDD), U2.39 (DVDD), U2.6 (DVDD), TP6.1; no longer L1.1
- net +3V3: now also TP4.1
- net D+: now also U3.4 (I/O2); no longer J1.A6 (D+), J1.B6 (D+)
- net D-: now also U3.6 (I/O1); no longer J1.A7 (D-), J1.B7 (D-)
- net GND: now also C19.2, TP2.1, U3.2 (GND)
- net SWCLK: now also TP1.1
- net SWD: now also TP3.1
- net VBUS: now also C19.1, TP5.1, U3.5 (VBUS)
- net VREG_LX: now also L1.1; no longer L1.2
- new net USB_D+: J1.A6 (D+), J1.B6 (D+), U3.3 (I/O2)
- new net USB_D-: J1.A7 (D-), J1.B7 (D-), U3.1 (I/O1)
Other:
- moved on the sheet: C1, C10, C11, C12, C13, C14, C15, C16, C17, C18, C2, C3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

Commit message: uwu nyaaa puurs at you
Parts:
- added C20, C21, C22: 4.7u, Capacitor_SMD:C_0402_1005Metric, symbol Device:C
- added NT1: NetTie_2, NetTie:NetTie-2_SMD_Pad2.0mm, symbol Device:NetTie_2
- J1: value C52209111 -> C2765186; footprint easyeda2kicad:USB-SMD_HH-16P-TYPE-C-Y495 -> HavenPCB:USB-C-SMD_TYPE-C-16PIN-2MD-073
Connections:
- net +1V1: now also C22.1
- net +3V3: now also C21.1
- net GND: now also C20.2, C21.2, C22.2, NT1.2; no longer C6.2, C7.2, U2.47 (VREG_PGND)
- net VBUS: now also C20.1
- net RP_D-: now reaches R6.2, U2.51 (USB_DM)
- net RP_D+: now reaches R7.2, U2.52 (USB_DP)
- new net VREG_GND: C6.2, C7.2, NT1.1, U2.47 (VREG_PGND)

Commit message: dsafanjkhf
Parts:
- added SW2: Up, Button_Switch_THT:SW_PUSH_6mm_H5mm, symbol Switch:SW_Push
- added SW3: Right, Button_Switch_THT:SW_PUSH_6mm_H5mm, symbol Switch:SW_Push
- added SW4: Left, Button_Switch_THT:SW_PUSH_6mm_H5mm, symbol Switch:SW_Push
- added SW5: Down, Button_Switch_THT:SW_PUSH_6mm_H5mm, symbol Switch:SW_Push
- added SW6: X, Button_Switch_THT:SW_PUSH_6mm_H5mm, symbol Switch:SW_Push
- added SW7: Y, Button_Switch_THT:SW_PUSH_6mm_H5mm, symbol Switch:SW_Push
- added SW8: B, Button_Switch_THT:SW_PUSH_6mm_H5mm, symbol Switch:SW_Push
- added SW9: A, Button_Switch_THT:SW_PUSH_6mm_H5mm, symbol Switch:SW_Push
Connections:
- net GND: now also SW2.2, SW3.2, SW4.2, SW5.2, SW6.2, SW7.2, SW8.2, SW9.2
- net Down: now reaches U2.13 (GPIO9)
- net Down: now also SW5.1
- net Right: now reaches U2.14 (GPIO10)
- net Right: now also SW3.1
- net Y: now reaches U2.32 (GPIO20)
- net Y: now also SW7.1
- net B: now reaches U2.33 (GPIO21)
- net B: now also SW8.1
- net A: now reaches U2.34 (GPIO22)
- net A: now also SW9.1
- net X: now reaches U2.35 (GPIO23)
- net X: now also SW6.1
- net Up: now reaches U2.7 (GPIO4)
- net Up: now also SW2.1
- net Left: now reaches U2.8 (GPIO5)
- net Left: now also SW4.1

Commit message: final
Parts:
- removed C20, C21: 4.7u, Capacitor_SMD:C_0402_1005Metric, symbol Device:C
- removed TP1, TP2, TP3, TP4, TP5, TP6: TestPoint, TestPoint:TestPoint_Pad_D1.5mm, symbol Connector:TestPoint
Connections:
- net +1V1: no longer C22.1
